Commit message: fix: align D405 views with gripper direction

File: Rviz/src/franzi_description/urdf/wheel_robot_4.0.urdf (robot description, URDF)
Before this commit: robot wheel_robot_4.0, 37 links, 36 joints
Joints:
- joint left_wrist_d405_joint: origin xyz=-0.0301 0.057975 -0.13418 rpy=3.1416 0 0 -> xyz=-0.0301 0.057975 -0.13418 rpy=0 0 0
- joint right_wrist_d405_joint: origin xyz=-0.0301 -0.057975 -0.13418 rpy=3.1416 0 0 -> xyz=-0.0301 -0.057975 -0.13418 rpy=0 0 0
