Commit message: update the franzi model to the wheel_robot_26.8.16_3 export
Re-export from SolidWorks. franzi_description and franzi_moveit_config only;
franzi_pick_place and IssacSim still name the old links and are left for a
follow-up.

URDF (franzi_description):
- rename wheel_robot_4.0 -> wheel_robot_26.8.16_3 across both packages
- the export's root is not REP-103 (robot stands along +X): the exported root
  is renamed base_body_Link and a massless base_link carrying the inverse
  permutation is put in front of it, keeping the origin and orientation the
  previous model and task.yaml measure against
- port the hand-authored SDK flange/TCP frames: wrist_roll_Link is now the
  flange frame itself, so each *_tcp hangs 273.5 mm along wrist_roll +x
- link renames: leftfinger1/2_Link -> left_finger01/02_Link, left_wrist_d405
  -> left_D405 (+ right); new left/right_j0_Link and left/right_gripper mount
- shoulder_pitch and elbow_pitch limits changed sign
- all 43 meshes replaced; 6 obsolete meshes removed
- add README.md and scripts/check_description.py (FK-based geometry checks)

MoveIt (franzi_moveit_config):
- SRDF/xacro renamed; collision matrix follows the new tree (base_body_Link,
  j0, gripper_link); finger01<->finger02 disabled so "closed" is
  collision-free
- gripper open/closed states recomputed: 95 mm open, 0 mm closed both sides
- joint_limits, moveit_controllers, demo publisher take the new finger names
- add scripts/check_moveit_config.py (RobotModel load + named-state collisions)

Verified: both packages build; check_description.py and check_moveit_config.py
pass; MoveIt RobotModel loads and every named state is self-collision-free.

Co-Authored-By: Claude Sonnet 5 <noreply@anthropic.com>
Claude-Session: https://claude.ai/code/session_01NQg1yaEuq2SPJPfnfuQ4ks

File: Rviz/src/franzi_description/urdf/wheel_robot_26.8.16_3.urdf (robot description, URDF)
Before this commit: robot wheel_robot_4.0, 37 links, 36 joints
Links:
- removed link left_wrist_d405_Link
- removed link leftfinger1_Link
- removed link leftfinger2_Link
- removed link right_wrist_d405_Link
- removed link rightfinger1_Link
- removed link rightfinger2_Link
- added link base_body_Link, mass 61.5; collision mesh filename=package://franzi_description/meshes/base_link.STL; visual mesh filename=package://franzi_description/meshes/base_link.STL
- added link left_D405_Link, mass 0.1; collision mesh filename=package://franzi_description/meshes/left_D405_Link.STL; visual mesh filename=package://franzi_description/meshes/left_D405_Link.STL
- added link left_finger01_Link, mass 0.1; collision mesh filename=package://franzi_description/meshes/left_finger01_Link.STL; visual mesh filename=package://franzi_description/meshes/left_finger01_Link.STL
- added link left_finger02_Link, mass 0.1; collision mesh filename=package://franzi_description/meshes/left_finger02_Link.STL; visual mesh filename=package://franzi_description/meshes/left_finger02_Link.STL
- added link left_flange
- added link left_gripper_link, mass 0.5; collision mesh filename=package://franzi_description/meshes/left_gripper_link.STL; visual mesh filename=package://franzi_description/meshes/left_gripper_link.STL
- added link left_j0_Link, mass 0.3; collision mesh filename=package://franzi_description/meshes/left_j0_Link.STL; visual mesh filename=package://franzi_description/meshes/left_j0_Link.STL
- added link left_tcp
- added link right_D405_Link, mass 0.1; collision mesh filename=package://franzi_description/meshes/right_D405_Link.STL; visual mesh filename=package://franzi_description/meshes/right_D405_Link.STL
- added link right_finger01_Link, mass 0.1; collision mesh filename=package://franzi_description/meshes/right_finger01_Link.STL; visual mesh filename=package://franzi_description/meshes/right_finger01_Link.STL
- added link right_finger02_Link, mass 0.1; collision mesh filename=package://franzi_description/meshes/right_finger02_Link.STL; visual mesh filename=package://franzi_description/meshes/right_finger02_Link.STL
- added link right_flange
- added link right_gripper_Link, mass 0.5; collision mesh filename=package://franzi_description/meshes/right_gripper_Link.STL; visual mesh filename=package://franzi_description/meshes/right_gripper_Link.STL
- added link right_j0_Link, mass 0.3; collision mesh filename=package://franzi_description/meshes/right_j0_Link.STL; visual mesh filename=package://franzi_description/meshes/right_j0_Link.STL
- added link right_tcp
- link base_link: mass 61.5 -> None; geometry 
- link left_wrist_roll_Link: mass 1.5 -> 1
- link right_wrist_roll_Link: mass 1.5 -> 1
Joints:
- removed joint left_wrist_d405_joint
- removed joint leftfinger1_joint
- removed joint leftfinger2_joint
- removed joint right_wrist_d405_joint
- removed joint rightfinger1_joint
- removed joint rightfinger2_joint
- added joint base_frame_joint: type fixed, parent base_link, child base_body_Link, origin xyz=0 0 0.24785 rpy=0 -1.57079632679 -1.57079632679
- added joint left_D405_joint: type fixed, parent left_gripper_link, child left_D405_Link, origin xyz=0.062698 0 0.0248 rpy=0 0 0, axis 0 0 0
- added joint left_finger01_joint: type prismatic, parent left_gripper_link, child left_finger01_Link, origin xyz=-0.00175 0.0476 0.17004 rpy=-1.5708 0 0, axis 0 0 1, limit lower=-0.0475 upper=0 effort=100 velocity=0.1
- added joint left_finger02_joint: type prismatic, parent left_gripper_link, child left_finger02_Link, origin xyz=-0.00175 -0.0474 0.17004 rpy=-1.5708 0 0, axis 0 0 1, limit lower=0 upper=0.0475 effort=100 velocity=0.1
- added joint left_flange_joint: type fixed, parent left_wrist_roll_Link, child left_flange, origin xyz=0 0 0 rpy=0 0 0
- added joint left_gripper_joint: type fixed, parent left_wrist_roll_Link, child left_gripper_link, origin xyz=0.0825 0 0 rpy=0 -1.5708 -3.14, axis 0 0 0, limit lower=0 upper=0.0475 effort=100 velocity=3.14
- added joint left_j0_joint: type fixed, parent torso_Link, child left_j0_Link, origin xyz=0 0.2385 0.3897 rpy=1.5708 1.5708 0, axis 0 0 0
- added joint left_tcp_joint: type fixed, parent left_flange, child left_tcp, origin xyz=0.2735 0 0 rpy=-1.57079632679 0 0
- added joint right_D405_joint: type fixed, parent right_gripper_Link, child right_D405_Link, origin xyz=0.062698 0 0.025 rpy=0 0 0, axis 0 0 0
- added joint right_finger01_joint: type prismatic, parent right_gripper_Link, child right_finger01_Link, origin xyz=-0.00175 -0.0474 0.16994 rpy=-1.5708 0 0, axis 0 0 1, limit lower=0 upper=0.0475 effort=0 velocity=0
- added joint right_finger02_joint: type prismatic, parent right_gripper_Link, child right_finger02_Link, origin xyz=-0.00175 0.0476 0.16994 rpy=-1.5708 0 0, axis 0 0 1, limit lower=-0.0475 upper=0 effort=0 velocity=0
- added joint right_flange_joint: type fixed, parent right_wrist_roll_Link, child right_flange, origin xyz=0 0 0 rpy=0 0 0
- added joint right_gripper_joint: type fixed, parent right_wrist_roll_Link, child right_gripper_Link, origin xyz=0.0824 0 0 rpy=0 -1.5708 3.14, axis 0 0 0, limit lower=0 upper=0.0475 effort=100 velocity=3.14
- added joint right_j0_joint: type fixed, parent torso_Link, child right_j0_Link, origin xyz=0 -0.2385 0.3897 rpy=1.5708 1.5708 0, axis 0 0 0
- added joint right_tcp_joint: type fixed, parent right_flange, child right_tcp, origin xyz=0.2735 0 0 rpy=1.57079632679 0 0
- joint 2Dlidar_joint: origin xyz=-0.22 -0.19 0.2474 rpy=0 0 0 -> xyz=-0.00045298 -0.22 -0.19 rpy=1.5708 0 1.5708; parent base_link -> base_body_Link
- joint MID360_joint: origin xyz=0.0765 0.1954 0.24623 rpy=0 0 0 -> xyz=-0.0016259 0.0765 0.1954 rpy=1.5708 0 1.5708; parent base_link -> base_body_Link
- joint body_d435_joint: origin xyz=0.10174 0.0175 0.23507 rpy=3.1416 0.87128 3.1416 -> xyz=0.10174 0.0175 0.25077 rpy=2.2703 0 1.5708
- joint calf_pitch_joint: axis 0 1 0 -> 0 0 1; origin xyz=0 0 0.24785 rpy=0 0 0 -> xyz=0 0 0 rpy=0 0 0; parent base_link -> base_body_Link
- joint head_d435_joint: origin xyz=0.092208 0.0175 0.15141 rpy=-3.1416 1.2217 3.1416 -> xyz=0.15141 0.092208 0.0175 rpy=-2.7925 -1.5708 1.5708
- joint head_pitch_joint: axis 0 1 0 -> 0 0 1; origin xyz=0 0 0.063 rpy=0 0 0 -> xyz=0 0 0.063 rpy=1.5708 -1.5708 0
- joint head_yaw_joint: origin xyz=0 0 0.461 rpy=0 0 0 -> xyz=0 0 0.4767 rpy=0 0 3.14
- joint left_elbow_pitch_joint: axis 0 1 0 -> 0 0 1; limit lower=-2.62 upper=0.13 effort=100 velocity=3.14 -> lower=-0.26 upper=2.62 effort=100 velocity=3.14; origin xyz=0.017 0 -0.145 rpy=0 0 0 -> xyz=-0.017 0 0 rpy=1.5708 0 0
- joint left_front_steering_joint: origin xyz=0.13 0.213 0.1114 rpy=0 0 0 -> xyz=-0.13645 0.13 0.213 rpy=1.5708 0 1.5708; parent base_link -> base_body_Link
- joint left_shoulder_pitch_joint: axis 0 1 0 -> 0 0 1; limit lower=-3.489 upper=2.617 effort=100 velocity=3.14 -> lower=-2.617 upper=3.489 effort=100 velocity=3.14; origin xyz=0 0.166 0.374 rpy=0 0 0 -> xyz=0 0 0 rpy=0 0 0; parent torso_Link -> left_j0_Link
- joint left_shoulder_roll_joint: axis 1 0 0 -> 0 0 1; origin xyz=0 0.0725 0 rpy=0 0 0 -> xyz=0 0 0 rpy=-1.5708 -1.5708 0
- joint left_shoulder_yaw_joint: origin xyz=0 0 -0.118 rpy=0 0 0 -> xyz=0 0.263 0 rpy=-1.5708 1.5708 0
- joint left_wrist_pitch_joint: axis 0 1 0 -> 0 0 1; origin xyz=0 0 -0.1658 rpy=0 0 0 -> xyz=0 0 0 rpy=1.5708 -1.5708 0
- joint left_wrist_roll_joint: axis 1 0 0 -> 0 0 1; origin xyz=0.0303 0 0 rpy=0 0 0 -> xyz=0 0 0 rpy=-1.5708 0 0
- joint left_wrist_yaw_joint: origin xyz=-0.017 0 -0.1262 rpy=0 0 0 -> xyz=0.017 0.292 0 rpy=-1.5708 0 0
- joint rear_steering_joint: origin xyz=-0.255 0 0.1054 rpy=0 0 0 -> xyz=-0.14245 -0.255 0 rpy=1.5708 0 1.5708; parent base_link -> base_body_Link
- joint right_elbow_pitch_joint: axis 0 1 0 -> 0 0 1; limit lower=-2.62 upper=0.13 effort=100 velocity=3.14 -> lower=-0.26 upper=2.62 effort=100 velocity=3.14; origin xyz=0.017 0 -0.145 rpy=0 0 0 -> xyz=-0.017 0 0 rpy=1.5708 0 0
- joint right_front_steering_joint: origin xyz=0.13 -0.213 0.1114 rpy=0 0 0 -> xyz=-0.13645 0.13 -0.213 rpy=1.5708 0 1.5708; parent base_link -> base_body_Link
- joint right_shoulder_pitch_joint: axis 0 1 0 -> 0 0 1; limit lower=-3.489 upper=2.617 effort=100 velocity=3.14 -> lower=-2.617 upper=3.489 effort=100 velocity=3.14; origin xyz=0 -0.166 0.374 rpy=0 0 0 -> xyz=0 0 0 rpy=0 0 0; parent torso_Link -> right_j0_Link
- joint right_shoulder_roll_joint: axis 1 0 0 -> 0 0 1; origin xyz=0 -0.0725 0 rpy=0 0 0 -> xyz=0 0 0 rpy=-1.5708 -1.5708 0
- joint right_shoulder_yaw_joint: origin xyz=0 0 -0.118 rpy=0 0 0 -> xyz=0 0.263 0 rpy=-1.5708 1.5708 0
- joint right_wrist_pitch_joint: axis 0 1 0 -> 0 0 1; origin xyz=0 0 -0.1658 rpy=0 0 0 -> xyz=0 0 0 rpy=1.5708 -1.5708 0
- joint right_wrist_roll_joint: axis 1 0 0 -> 0 0 1; origin xyz=0.0303 0 0 rpy=0 0 0 -> xyz=0 0 0 rpy=-1.5708 0 0
- joint right_wrist_yaw_joint: origin xyz=-0.017 0 -0.1262 rpy=0 0 0 -> xyz=0.017 0.292 0 rpy=-1.5708 0 0
- joint thigh_pitch_joint: axis 0 1 0 -> 0 0 1; origin xyz=0 0 0.3 rpy=0 0 0 -> xyz=0.3 0 0 rpy=0 0 0
- joint waist_pitch_joint: axis 0 1 0 -> 0 0 1; limit lower=-0.5235 upper=0.5235 effort=100 velocity=3.14 -> lower=-1.31 upper=0.5235 effort=100 velocity=3.14; origin xyz=0 0 0.35 rpy=0 0 0 -> xyz=0.35 0 0 rpy=0 0 1.5708
- joint waist_yaw_joint: origin xyz=0 0 0.0807 rpy=0 0 0 -> xyz=0 -0.065 0 rpy=1.5708 0 0

File: Rviz/src/franzi_moveit_config/config/wheel_robot_26.8.16_3.urdf.xacro (robot description, xacro)
@@ -1,7 +1,7 @@
 <?xml version="1.0"?>
-<robot xmlns:xacro="http://www.ros.org/wiki/xacro" name="wheel_robot_4.0">
+<robot xmlns:xacro="http://www.ros.org/wiki/xacro" name="wheel_robot_26.8.16_3">
   <!-- Keep the source description unchanged and add a massless root only for
        KDL, which cannot represent inertia on the root link. -->
-  <xacro:include filename="$(find franzi_description)/urdf/wheel_robot_4.0.urdf"/>
+  <xacro:include filename="$(find franzi_description)/urdf/wheel_robot_26.8.16_3.urdf"/>
   <link name="moveit_root"/>
   <joint name="moveit_root_joint" type="fixed">
